Commit message: Perseverance URDF (from OnShape) (#3)

File: perseverance/urdf/rover.urdf.xacro (robot description, xacro)
@@ -1,21 +1,53 @@
 <?xml version="1.0" ?>
 <!-- Generated using onshape-to-robot -->
-<!-- Onshape https://cad.onshape.com/documents/31ca51e87164d5a2ae3b11dc/w/1e07aa3f18f08d453ac8b6a1/e/c6031188983b3698192fd890 -->
+<!-- Onshape https://cad.onshape.com/documents/31ca51e87164d5a2ae3b11dc/w/1e07aa3f18f08d453ac8b6a1/e/be108145cc25fea61866c58d -->
 <robot name="perseverance" xmlns:xacro="http://ros.org/wiki/xacro">
   <xacro:property name="mesh_dir" value="file://$(find perseverance)/meshes"/>
-  <!-- Link base -->
+  <!-- Link base_link -->
   <link name="base_link">
     <inertial>
-      <origin xyz="0.00194388 -0.00615083 0.0142334" rpy="0 0 0"/>
-      <mass value="0.792684"/>
-      <inertia ixx="0.0056261" ixy="-0.000184338" ixz="-4.5498e-06" iyy="0.00337652" iyz="3.08805e-05" izz="0.00873301"/>
-    </inertial>
+      <origin xyz="0.00132088 -0.0106351 0.0110544" rpy="0 0 0"/>
+      <mass value="1.16655"/>
+      <inertia ixx="0.00718086" ixy="-0.000191247" ixz="-9.44893e-06" iyy="0.00962338" iyz="0.000134967" izz="0.0161498"/>
+    </inertial>
+    <!-- Part rightbogie -->
+    <visual>
+      <origin xyz="-0.15 0.0418583 -0.00306575" rpy="0 -0 -1.5708"/>
+      <geometry>
+        <mesh filename="${mesh_dir}/rightbogie.stl"/>
+      </geometry>
+      <material name="rightbogie_material">
+        <color rgba="0.262745 0.282353 0.301961 1"/>
+      </material>
+    </visual>
+    <collision>
+      <origin xyz="-0.15 0.0418583 -0.00306575" rpy="0 -0 -1.5708"/>
+      <geometry>
+        <mesh filename="${mesh_dir}/rightbogie.stl"/>
+      </geometry>
+    </collision>
+    <!-- Part bevel_0_85m_18t_45deg -->
+    <visual>
+      <origin xyz="-0.012226 -0.042 0.024" rpy="-0 1.5708 0"/>
+      <geometry>
+        <mesh filename="${mesh_dir}/bevel_0_85m_18t_45deg.stl"/>
+      </geometry>
+      <material name="bevel_0_85m_18t_45deg_material">
+        <color rgba="0.729412 0.25098 0.105882 1"/>
+      </material>
+    </visual>
+    <collision>
+      <origin xyz="-0.012226 -0.042 0.024" rpy="-0 1.5708 0"/>
+      <geometry>
+        <mesh filename="${mesh_dir}/bevel_0_85m_18t_45deg.stl"/>
+      </geometry>
+    </collision>
     <!-- Part base_link -->
     <visual>
       <origin xyz="0 0 0" rpy="0 -0 0"/>
       <geometry>
-        <mesh filename="${mesh_dir}/body.stl"/>
-      </geometry>
-      <material name="body_material">
+        <mesh filename="${mesh_dir}/base_link.stl"/>
+      </geometry>
+      <material name="base_link_material">
         <color rgba="0.811765 0.858824 0.898039 1"/>
       </material>
@@ -24,7 +56,455 @@
       <origin xyz="0 0 0" rpy="0 -0 0"/>
       <geometry>
-        <mesh filename="${mesh_dir}/body.stl"/>
-      </geometry>
-    </collision>
-  </link>
+        <mesh filename="${mesh_dir}/base_link.stl"/>
+      </geometry>
+    </collision>
+    <!-- Part bevel_0_85m_18t_45deg_2 -->
+    <visual>
+      <origin xyz="0.012226 -0.042 0.024" rpy="-1.3494e-79 -1.5708 0"/>
+      <geometry>
+        <mesh filename="${mesh_dir}/bevel_0_85m_18t_45deg.stl"/>
+      </geometry>
+      <material name="bevel_0_85m_18t_45deg_2_material">
+        <color rgba="0.729412 0.25098 0.105882 1"/>
+      </material>
+    </visual>
+    <collision>
+      <origin xyz="0.012226 -0.042 0.024" rpy="-1.3494e-79 -1.5708 0"/>
+      <geometry>
+        <mesh filename="${mesh_dir}/bevel_0_85m_18t_45deg.stl"/>
+      </geometry>
+    </collision>
+    <!-- Part mg995 -->
+    <visual>
+      <origin xyz="-0.1425 -0.140031 0.043" rpy="3.14159 -0 -3.14159"/>
+      <geometry>
+        <mesh filename="${mesh_dir}/mg995.stl"/>
+      </geometry>
+      <material name="mg995_material">
+        <color rgba="0.792157 0.819608 0.933333 1"/>
+      </material>
+    </visual>
+    <collision>
+      <origin xyz="-0.1425 -0.140031 0.043" rpy="3.14159 -0 -3.14159"/>
+      <geometry>
+        <mesh filename="${mesh_dir}/mg995.stl"/>
+      </geometry>
+    </collision>
+    <!-- Part mg995_2 -->
+    <visual>
+      <origin xyz="-0.150764 0.100122 0.0432278" rpy="3.14159 -0 1.74533"/>
+      <geometry>
+        <mesh filename="${mesh_dir}/mg995.stl"/>
+      </geometry>
+      <material name="mg995_2_material">
+        <color rgba="0.792157 0.819608 0.933333 1"/>
+      </material>
+    </visual>
+    <collision>
+      <origin xyz="-0.150764 0.100122 0.0432278" rpy="3.14159 -0 1.74533"/>
+      <geometry>
+        <mesh filename="${mesh_dir}/mg995.stl"/>
+      </geometry>
+    </collision>
+    <!-- Part mg995_3 -->
+    <visual>
+      <origin xyz="0.1425 -0.140031 0.043" rpy="3.14159 -0 -2.01228e-16"/>
+      <geometry>
+        <mesh filename="${mesh_dir}/mg995.stl"/>
+      </geometry>
+      <material name="mg995_3_material">
+        <color rgba="0.792157 0.819608 0.933333 1"/>
+      </material>
+    </visual>
+    <collision>
+      <origin xyz="0.1425 -0.140031 0.043" rpy="3.14159 -0 -2.01228e-16"/>
+      <geometry>
+        <mesh filename="${mesh_dir}/mg995.stl"/>
+      </geometry>
+    </collision>
+    <!-- Part leftrocker -->
+    <visual>
+      <origin xyz="0.115 -0.042 0.024" rpy="0 -0 -1.5708"/>
+      <geometry>
+        <mesh filename="${mesh_dir}/leftrocker.stl"/>
+      </geometry>
+      <material name="leftrocker_material">
+        <color rgba="0.262745 0.282353 0.301961 1"/>
+      </material>
+    </visual>
+    <collision>
+      <origin xyz="0.115 -0.042 0.024" rpy="0 -0 -1.5708"/>
+      <geometry>
+        <mesh filename="${mesh_dir}/leftrocker.stl"/>
+      </geometry>
+    </collision>
+    <!-- Part rightrocker -->
+    <visual>
+      <origin xyz="-0.115 -0.042 0.024" rpy="0 -0 -1.5708"/>
+      <geometry>
+        <mesh filename="${mesh_dir}/rightrocker.stl"/>
+      </geometry>
+      <material name="rightrocker_material">
+        <color rgba="0.262745 0.282353 0.301961 1"/>
+      </material>
+    </visual>
+    <collision>
+      <origin xyz="-0.115 -0.042 0.024" rpy="0 -0 -1.5708"/>
+      <geometry>
+        <mesh filename="${mesh_dir}/rightrocker.stl"/>
+      </geometry>
+    </collision>
+    <!-- Part mg995_4 -->
+    <visual>
+      <origin xyz="0.150764 0.100122 0.0432278" rpy="3.14159 -0 1.39626"/>
+      <geometry>
+        <mesh filename="${mesh_dir}/mg995.stl"/>
+      </geometry>
+      <material name="mg995_4_material">
+        <color rgba="0.792157 0.819608 0.933333 1"/>
+      </material>
+    </visual>
+    <collision>
+      <origin xyz="0.150764 0.100122 0.0432278" rpy="3.14159 -0 1.39626"/>
+      <geometry>
+        <mesh filename="${mesh_dir}/mg995.stl"/>
+      </geometry>
+    </collision>
+    <!-- Part leftbogie -->
+    <visual>
+      <origin xyz="0.15 0.0418583 -0.00306575" rpy="0 -0 -1.5708"/>
+      <geometry>
+        <mesh filename="${mesh_dir}/leftbogie.stl"/>
+      </geometry>
+      <material name="leftbogie_material">
+        <color rgba="0.262745 0.282353 0.301961 1"/>
+      </material>
+    </visual>
+    <collision>
+      <origin xyz="0.15 0.0418583 -0.00306575" rpy="0 -0 -1.5708"/>
+      <geometry>
+        <mesh filename="${mesh_dir}/leftbogie.stl"/>
+      </geometry>
+    </collision>
+  </link>
+  <!-- Link rearsteeringarm -->
+  <link name="rearsteeringarm">
+    <inertial>
+      <origin xyz="0.0162576 1.99588e-09 -0.0222692" rpy="0 0 0"/>
+      <mass value="0.0309807"/>
+      <inertia ixx="1.46169e-05" ixy="-1.34476e-13" ixz="1.19558e-06" iyy="1.75736e-05" iyz="1.92805e-12" izz="5.44298e-06"/>
+    </inertial>
+    <!-- Part rearsteeringarm -->
+    <visual>
+      <origin xyz="2.77556e-17 2.77556e-17 -0.005" rpy="9.24446e-33 -2.82529e-32 -4.77087e-18"/>
+      <geometry>
+        <mesh filename="${mesh_dir}/rearsteeringarm.stl"/>
+      </geometry>
+      <material name="rearsteeringarm_material">
+        <color rgba="0.458824 0.105882 0 1"/>
+      </material>
+    </visual>
+    <collision>
+      <origin xyz="2.77556e-17 2.77556e-17 -0.005" rpy="9.24446e-33 -2.82529e-32 -4.77087e-18"/>
+      <geometry>
+        <mesh filename="${mesh_dir}/rearsteeringarm.stl"/>
+      </geometry>
+    </collision>
+  </link>
+  <!-- Link wheelhub -->
+  <link name="wheelhub">
+    <inertial>
+      <origin xyz="-3.19312e-19 3.11997e-18 0.00460287" rpy="0 0 0"/>
+      <mass value="0.0820664"/>
+      <inertia ixx="3.08808e-05" ixy="-3.64091e-55" ixz="-1.42616e-21" iyy="3.08808e-05" iyz="1.12352e-54" izz="5.62507e-05"/>
+    </inertial>
+    <!-- Part wheelhub -->
+    <visual>
+      <origin xyz="0 0 -0.005" rpy="-1.5708 1.35456e-17 3.31859e-65"/>
+      <geometry>
+        <mesh filename="${mesh_dir}/wheelhub.stl"/>
+      </geometry>
+      <material name="wheelhub_material">
+        <color rgba="0.498039 0.498039 0.498039 1"/>
+      </material>
+    </visual>
+    <collision>
+      <origin xyz="0 0 -0.005" rpy="-1.5708 1.35456e-17 3.31859e-65"/>
+      <geometry>
+        <mesh filename="${mesh_dir}/wheelhub.stl"/>
+      </geometry>
+    </collision>
+  </link>
+  <!-- Joint from rearsteeringarm to wheelhub -->
+  <joint name="bl_wheel" type="continuous">
+    <origin xyz="-0.005 -5.55112e-17 -0.0463814" rpy="-1.5708 1.249e-16 -1.5708"/>
+    <parent link="rearsteeringarm"/>
+    <child link="wheelhub"/>
+    <axis xyz="0 0 1"/>
+    <limit effort="10" velocity="10"/>
+  </joint>
+  <!-- Joint from base_link to rearsteeringarm -->
+  <joint name="bl_steering" type="revolute">
+    <origin xyz="0.1525 0.10997 -0.00127218" rpy="-1.249e-16 4.18641e-16 2.96706"/>
+    <parent link="base_link"/>
+    <child link="rearsteeringarm"/>
+    <axis xyz="0 0 1"/>
+    <limit effort="10" velocity="10" lower="-0.610865" upper="0.610865"/>
+  </joint>
+  <!-- Link rearsteeringarm_2 -->
+  <link name="rearsteeringarm_2">
+    <inertial>
+      <origin xyz="0.0162576 1.99588e-09 -0.0222692" rpy="0 0 0"/>
+      <mass value="0.0309807"/>
+      <inertia ixx="1.46169e-05" ixy="-1.34476e-13" ixz="1.19558e-06" iyy="1.75736e-05" iyz="1.92805e-12" izz="5.44298e-06"/>
+    </inertial>
+    <!-- Part rearsteeringarm_2 -->
+    <visual>
+      <origin xyz="2.77556e-17 2.77556e-17 -0.005" rpy="-8.84344e-75 -0 -7.75341e-18"/>
+      <geometry>
+        <mesh filename="${mesh_dir}/rearsteeringarm.stl"/>
+      </geometry>
+      <material name="rearsteeringarm_2_material">
+        <color rgba="0.458824 0.105882 0 1"/>
+      </material>
+    </visual>
+    <collision>
+      <origin xyz="2.77556e-17 2.77556e-17 -0.005" rpy="-8.84344e-75 -0 -7.75341e-18"/>
+      <geometry>
+        <mesh filename="${mesh_dir}/rearsteeringarm.stl"/>
+      </geometry>
+    </collision>
+  </link>
+  <!-- Link wheelhub_2 -->
+  <link name="wheelhub_2">
+    <inertial>
+      <origin xyz="2.74897e-17 3.11997e-18 0.00460287" rpy="0 0 0"/>
+      <mass value="0.0820664"/>
+      <inertia ixx="3.08808e-05" ixy="3.5356e-93" ixz="-7.5456e-22" iyy="3.08808e-05" iyz="5.5184e-80" izz="5.62507e-05"/>
+    </inertial>
+    <!-- Part wheelhub_2 -->
+    <visual>
+      <origin xyz="2.77556e-17 0 -0.005" rpy="-1.5708 1.93111e-18 9.91647e-75"/>
+      <geometry>
+        <mesh filename="${mesh_dir}/wheelhub.stl"/>
+      </geometry>
+      <material name="wheelhub_2_material">
+        <color rgba="0.498039 0.498039 0.498039 1"/>
+      </material>
+    </visual>
+    <collision>
+      <origin xyz="2.77556e-17 0 -0.005" rpy="-1.5708 1.93111e-18 9.91647e-75"/>
+      <geometry>
+        <mesh filename="${mesh_dir}/wheelhub.stl"/>
+      </geometry>
+    </collision>
+  </link>
+  <!-- Joint from rearsteeringarm_2 to wheelhub_2 -->
+  <joint name="br_wheel" type="continuous">
+    <origin xyz="-0.005 5.55112e-17 -0.0463814" rpy="1.5708 -0 1.5708"/>
+    <parent link="rearsteeringarm_2"/>
+    <child link="wheelhub_2"/>
+    <axis xyz="0 0 1"/>
+    <limit effort="10" velocity="10"/>
+  </joint>
+  <!-- Joint from base_link to rearsteeringarm_2 -->
+  <joint name="br_steering" type="revolute">
+    <origin xyz="-0.1525 0.10997 -0.00127218" rpy="4.22436e-59 -1.37735e-59 0.174533"/>
+    <parent link="base_link"/>
+    <child link="rearsteeringarm_2"/>
+    <axis xyz="0 0 1"/>
+    <limit effort="10" velocity="10" lower="-0.610865" upper="0.610865"/>
+  </joint>
+  <!-- Link frontsteeringarm -->
+  <link name="frontsteeringarm">
+    <inertial>
+      <origin xyz="0.0160954 1.24761e-09 -0.0207225" rpy="0 0 0"/>
+      <mass value="0.0305721"/>
+      <inertia ixx="1.28485e-05" ixy="-1.54012e-13" ixz="1.11198e-06" iyy="1.57606e-05" iyz="1.84212e-12" izz="5.35874e-06"/>
+    </inertial>
+    <!-- Part frontsteeringarm -->
+    <visual>
+      <origin xyz="0 0 -0.005" rpy="0 -0 9.24446e-33"/>
+      <geometry>
+        <mesh filename="${mesh_dir}/frontsteeringarm.stl"/>
+      </geometry>
+      <material name="frontsteeringarm_material">
+        <color rgba="0.458824 0.105882 0 1"/>
+      </material>
+    </visual>
+    <collision>
+      <origin xyz="0 0 -0.005" rpy="0 -0 9.24446e-33"/>
+      <geometry>
+        <mesh filename="${mesh_dir}/frontsteeringarm.stl"/>
+      </geometry>
+    </collision>
+  </link>
+  <!-- Link wheelhub_3 -->
+  <link name="wheelhub_3">
+    <inertial>
+      <origin xyz="-1.47254e-19 3.11997e-18 0.00460287" rpy="0 0 0"/>
+      <mass value="0.0820664"/>
+      <inertia ixx="3.08808e-05" ixy="0" ixz="-5.47239e-37" iyy="3.08808e-05" iyz="0" izz="5.62507e-05"/>
+    </inertial>
+    <!-- Part wheelhub_3 -->
+    <visual>
+      <origin xyz="0 0 -0.005" rpy="-1.5708 -2.15704e-32 0"/>
+      <geometry>
+        <mesh filename="${mesh_dir}/wheelhub.stl"/>
+      </geometry>
+      <material name="wheelhub_3_material">
+        <color rgba="0.498039 0.498039 0.498039 1"/>
+      </material>
+    </visual>
+    <collision>
+      <origin xyz="0 0 -0.005" rpy="-1.5708 -2.15704e-32 0"/>
+      <geometry>
+        <mesh filename="${mesh_dir}/wheelhub.stl"/>
+      </geometry>
+    </collision>
+  </link>
+  <!-- Joint from frontsteeringarm to wheelhub_3 -->
+  <joint name="fl_wheel" type="continuous">
+    <origin xyz="-0.005 -2.77556e-17 -0.0433189" rpy="-1.5708 -0 -1.5708"/>
+    <parent link="frontsteeringarm"/>
+    <child link="wheelhub_3"/>
+    <axis xyz="0 0 1"/>
+    <limit effort="10" velocity="10"/>
+  </joint>
+  <!-- Joint from base_link to frontsteeringarm -->
+  <joint name="fl_steering" type="revolute">
+    <origin xyz="0.1525 -0.140031 -0.0015" rpy="0 -0 3.14159"/>
+    <parent link="base_link"/>
+    <child link="frontsteeringarm"/>
+    <axis xyz="0 0 1"/>
+    <limit effort="10" velocity="10" lower="-0.610865" upper="0.610865"/>
+  </joint>
+  <!-- Link frontsteeringarm_2 -->
+  <link name="frontsteeringarm_2">
+    <inertial>
+      <origin xyz="-0.0160954 -1.24761e-09 -0.0207225" rpy="0 0 0"/>
+      <mass value="0.0305721"/>
+      <inertia ixx="1.28485e-05" ixy="-1.54012e-13" ixz="-1.11198e-06" iyy="1.57606e-05" iyz="-1.84212e-12" izz="5.35874e-06"/>
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