Commit message: new URDF file and meshes

File: perseverance/urdf/rover.urdf (robot description, URDF)
Before this commit: robot perseverance, 11 links, 10 joints
Links:
- removed link body
- removed link part_1
- removed link part_1_10
- removed link part_1_2
- removed link part_1_3
- removed link part_1_4
- removed link part_1_5
- removed link part_1_6
- removed link part_1_7
- removed link part_1_8
- removed link part_1_9
- added link base_link, mass 1.16655; collision mesh filename=package://meshes/base_link.stl; collision mesh filename=package://meshes/bevel_0_85m_18t_45deg.stl
- added link frontsteeringarm, mass 0.0305721; collision mesh filename=package://meshes/frontsteeringarm.stl; visual mesh filename=package://meshes/frontsteeringarm.stl
- added link frontsteeringarm_2, mass 0.0305721; collision mesh filename=package://meshes/frontsteeringarm.stl; visual mesh filename=package://meshes/frontsteeringarm.stl
- added link rearsteeringarm, mass 0.0309807; collision mesh filename=package://meshes/rearsteeringarm.stl; visual mesh filename=package://meshes/rearsteeringarm.stl
- added link rearsteeringarm_2, mass 0.0309807; collision mesh filename=package://meshes/rearsteeringarm.stl; visual mesh filename=package://meshes/rearsteeringarm.stl
- added link wheelhub, mass 0.0820664; collision mesh filename=package://meshes/wheelhub.stl; visual mesh filename=package://meshes/wheelhub.stl
- added link wheelhub_2, mass 0.0820664; collision mesh filename=package://meshes/wheelhub.stl; visual mesh filename=package://meshes/wheelhub.stl
- added link wheelhub_3, mass 0.0820664; collision mesh filename=package://meshes/wheelhub.stl; visual mesh filename=package://meshes/wheelhub.stl
- added link wheelhub_4, mass 0.0820664; collision mesh filename=package://meshes/wheelhub.stl; visual mesh filename=package://meshes/wheelhub.stl
- added link wheelhub_5, mass 0.0820664; collision mesh filename=package://meshes/wheelhub.stl; visual mesh filename=package://meshes/wheelhub.stl
- added link wheelhub_6, mass 0.0820664; collision mesh filename=package://meshes/wheelhub.stl; visual mesh filename=package://meshes/wheelhub.stl
Joints:
- joint bl_steering: child part_1 -> rearsteeringarm; parent body -> base_link
- joint bl_wheel: child part_1_2 -> wheelhub; parent part_1 -> rearsteeringarm
- joint br_steering: child part_1_3 -> rearsteeringarm_2; parent body -> base_link
- joint br_wheel: child part_1_4 -> wheelhub_2; parent part_1_3 -> rearsteeringarm_2
- joint fl_steering: child part_1_5 -> frontsteeringarm; parent body -> base_link
- joint fl_wheel: child part_1_6 -> wheelhub_3; parent part_1_5 -> frontsteeringarm
- joint fr_steering: child part_1_7 -> frontsteeringarm_2; parent body -> base_link
- joint fr_wheel: child part_1_8 -> wheelhub_4; parent part_1_7 -> frontsteeringarm_2
- joint ml_wheel: child part_1_10 -> wheelhub_6; parent body -> base_link
- joint mr_wheel: child part_1_9 -> wheelhub_5; parent body -> base_link

File: perseverance/urdf/rover.urdf.xacro (robot description, xacro)
@@ -3,11 +3,11 @@
 <!-- Onshape https://cad.onshape.com/documents/31ca51e87164d5a2ae3b11dc/w/1e07aa3f18f08d453ac8b6a1/e/be108145cc25fea61866c58d -->
 <robot name="perseverance" xmlns:xacro="http://ros.org/wiki/xacro">
-  <xacro:property name="mesh_dir" value="$(find-pkg-share perseverance)/meshes"/>
-  <!-- Link body -->
-  <link name="body">
+  <xacro:property name="mesh_dir" value="file://$(find perseverance)/meshes"/>
+  <!-- Link base_link -->
+  <link name="base_link">
     <inertial>
       <origin xyz="0.00132088 -0.0106351 0.0110544" rpy="0 0 0"/>
       <mass value="1.16655"/>
-      <!-- <inertia ixx="0.00718086" ixy="-0.000191247" ixz="-9.44893e-06" iyy="0.00962338" iyz="0.000134967" izz="0.0161498"/> -->
+      <inertia ixx="0.00718086" ixy="-0.000191247" ixz="-9.44893e-06" iyy="0.00962338" iyz="0.000134967" izz="0.0161498"/>
     </inertial>
     <!-- Part rightbogie -->
@@ -43,11 +43,11 @@
       </geometry>
     </collision>
-    <!-- Part body -->
+    <!-- Part base_link -->
     <visual>
       <origin xyz="0 0 0" rpy="0 -0 0"/>
       <geometry>
-        <mesh filename="${mesh_dir}/body.stl"/>
-      </geometry>
-      <material name="body_material">
+        <mesh filename="${mesh_dir}/base_link.stl"/>
+      </geometry>
+      <material name="base_link_material">
         <color rgba="0.811765 0.858824 0.898039 1"/>
       </material>
@@ -56,5 +56,5 @@
       <origin xyz="0 0 0" rpy="0 -0 0"/>
       <geometry>
-        <mesh filename="${mesh_dir}/body.stl"/>
+        <mesh filename="${mesh_dir}/base_link.stl"/>
       </geometry>
     </collision>
@@ -188,6 +188,6 @@
     </collision>
   </link>
-  <!-- Link part_1 -->
-  <link name="part_1">
+  <!-- Link rearsteeringarm -->
+  <link name="rearsteeringarm">
     <inertial>
       <origin xyz="0.0162576 1.99588e-09 -0.0222692" rpy="0 0 0"/>
@@ -195,11 +195,11 @@
       <inertia ixx="1.46169e-05" ixy="-1.34476e-13" ixz="1.19558e-06" iyy="1.75736e-05" iyz="1.92805e-12" izz="5.44298e-06"/>
     </inertial>
-    <!-- Part part_1 -->
+    <!-- Part rearsteeringarm -->
     <visual>
       <origin xyz="2.77556e-17 2.77556e-17 -0.005" rpy="9.24446e-33 -2.82529e-32 -4.77087e-18"/>
       <geometry>
-        <mesh filename="${mesh_dir}/part_1.stl"/>
-      </geometry>
-      <material name="part_1_material">
+        <mesh filename="${mesh_dir}/rearsteeringarm.stl"/>
+      </geometry>
+      <material name="rearsteeringarm_material">
         <color rgba="0.458824 0.105882 0 1"/>
       </material>
@@ -208,22 +208,22 @@
       <origin xyz="2.77556e-17 2.77556e-17 -0.005" rpy="9.24446e-33 -2.82529e-32 -4.77087e-18"/>
       <geometry>
-        <mesh filename="${mesh_dir}/part_1.stl"/>
-      </geometry>
-    </collision>
-  </link>
-  <!-- Link part_1_2 -->
-  <link name="part_1_2">
-    <inertial>
-      <origin xyz="-3.19312e-19 3.11998e-18 0.00460287" rpy="0 0 0"/>
+        <mesh filename="${mesh_dir}/rearsteeringarm.stl"/>
+      </geometry>
+    </collision>
+  </link>
+  <!-- Link wheelhub -->
+  <link name="wheelhub">
+    <inertial>
+      <origin xyz="-3.19312e-19 3.11997e-18 0.00460287" rpy="0 0 0"/>
       <mass value="0.0820664"/>
       <inertia ixx="3.08808e-05" ixy="-3.64091e-55" ixz="-1.42616e-21" iyy="3.08808e-05" iyz="1.12352e-54" izz="5.62507e-05"/>
     </inertial>
-    <!-- Part part_1_2 -->
+    <!-- Part wheelhub -->
     <visual>
       <origin xyz="0 0 -0.005" rpy="-1.5708 1.35456e-17 3.31859e-65"/>
       <geometry>
-        <mesh filename="${mesh_dir}/part_1__2.stl"/>
-      </geometry>
-      <material name="part_1_2_material">
+        <mesh filename="${mesh_dir}/wheelhub.stl"/>
+      </geometry>
+      <material name="wheelhub_material">
         <color rgba="0.498039 0.498039 0.498039 1"/>
       </material>
@@ -232,26 +232,26 @@
       <origin xyz="0 0 -0.005" rpy="-1.5708 1.35456e-17 3.31859e-65"/>
       <geometry>
-        <mesh filename="${mesh_dir}/part_1__2.stl"/>
-      </geometry>
-    </collision>
-  </link>
-  <!-- Joint from part_1 to part_1_2 -->
+        <mesh filename="${mesh_dir}/wheelhub.stl"/>
+      </geometry>
+    </collision>
+  </link>
+  <!-- Joint from rearsteeringarm to wheelhub -->
   <joint name="bl_wheel" type="continuous">
     <origin xyz="-0.005 -5.55112e-17 -0.0463814" rpy="-1.5708 1.249e-16 -1.5708"/>
-    <parent link="part_1"/>
-    <child link="part_1_2"/>
+    <parent link="rearsteeringarm"/>
+    <child link="wheelhub"/>
     <axis xyz="0 0 1"/>
     <limit effort="10" velocity="10"/>
   </joint>
-  <!-- Joint from body to part_1 -->
+  <!-- Joint from base_link to rearsteeringarm -->
   <joint name="bl_steering" type="revolute">
     <origin xyz="0.1525 0.10997 -0.00127218" rpy="-1.249e-16 4.18641e-16 2.96706"/>
-    <parent link="body"/>
-    <child link="part_1"/>
+    <parent link="base_link"/>
+    <child link="rearsteeringarm"/>
     <axis xyz="0 0 1"/>
     <limit effort="10" velocity="10" lower="-0.610865" upper="0.610865"/>
   </joint>
-  <!-- Link part_1_3 -->
-  <link name="part_1_3">
+  <!-- Link rearsteeringarm_2 -->
+  <link name="rearsteeringarm_2">
     <inertial>
       <origin xyz="0.0162576 1.99588e-09 -0.0222692" rpy="0 0 0"/>
@@ -259,11 +259,11 @@
       <inertia ixx="1.46169e-05" ixy="-1.34476e-13" ixz="1.19558e-06" iyy="1.75736e-05" iyz="1.92805e-12" izz="5.44298e-06"/>
     </inertial>
-    <!-- Part part_1_3 -->
+    <!-- Part rearsteeringarm_2 -->
     <visual>
       <origin xyz="2.77556e-17 2.77556e-17 -0.005" rpy="-8.84344e-75 -0 -7.75341e-18"/>
       <geometry>
-        <mesh filename="${mesh_dir}/part_1.stl"/>
-      </geometry>
-      <material name="part_1_3_material">
+        <mesh filename="${mesh_dir}/rearsteeringarm.stl"/>
+      </geometry>
+      <material name="rearsteeringarm_2_material">
         <color rgba="0.458824 0.105882 0 1"/>
       </material>
@@ -272,22 +272,22 @@
       <origin xyz="2.77556e-17 2.77556e-17 -0.005" rpy="-8.84344e-75 -0 -7.75341e-18"/>
       <geometry>
-        <mesh filename="${mesh_dir}/part_1.stl"/>
-      </geometry>
-    </collision>
-  </link>
-  <!-- Link part_1_4 -->
-  <link name="part_1_4">
-    <inertial>
-      <origin xyz="2.74897e-17 3.11998e-18 0.00460287" rpy="0 0 0"/>
+        <mesh filename="${mesh_dir}/rearsteeringarm.stl"/>
+      </geometry>
+    </collision>
+  </link>
+  <!-- Link wheelhub_2 -->
+  <link name="wheelhub_2">
+    <inertial>
+      <origin xyz="2.74897e-17 3.11997e-18 0.00460287" rpy="0 0 0"/>
       <mass value="0.0820664"/>
-      <inertia ixx="3.08808e-05" ixy="3.47568e-93" ixz="-7.5456e-22" iyy="3.08808e-05" iyz="5.5184e-80" izz="5.62507e-05"/>
-    </inertial>
-    <!-- Part part_1_4 -->
+      <inertia ixx="3.08808e-05" ixy="3.5356e-93" ixz="-7.5456e-22" iyy="3.08808e-05" iyz="5.5184e-80" izz="5.62507e-05"/>
+    </inertial>
+    <!-- Part wheelhub_2 -->
     <visual>
       <origin xyz="2.77556e-17 0 -0.005" rpy="-1.5708 1.93111e-18 9.91647e-75"/>
       <geometry>
-        <mesh filename="${mesh_dir}/part_1__2.stl"/>
-      </geometry>
-      <material name="part_1_4_material">
+        <mesh filename="${mesh_dir}/wheelhub.stl"/>
+      </geometry>
+      <material name="wheelhub_2_material">
         <color rgba="0.498039 0.498039 0.498039 1"/>
       </material>
@@ -296,26 +296,26 @@
       <origin xyz="2.77556e-17 0 -0.005" rpy="-1.5708 1.93111e-18 9.91647e-75"/>
       <geometry>
-        <mesh filename="${mesh_dir}/part_1__2.stl"/>
-      </geometry>
-    </collision>
-  </link>
-  <!-- Joint from part_1_3 to part_1_4 -->
+        <mesh filename="${mesh_dir}/wheelhub.stl"/>
+      </geometry>
+    </collision>
+  </link>
+  <!-- Joint from rearsteeringarm_2 to wheelhub_2 -->
   <joint name="br_wheel" type="continuous">
     <origin xyz="-0.005 5.55112e-17 -0.0463814" rpy="1.5708 -0 1.5708"/>
-    <parent link="part_1_3"/>
-    <child link="part_1_4"/>
+    <parent link="rearsteeringarm_2"/>
+    <child link="wheelhub_2"/>
     <axis xyz="0 0 1"/>
     <limit effort="10" velocity="10"/>
   </joint>
-  <!-- Joint from body to part_1_3 -->
+  <!-- Joint from base_link to rearsteeringarm_2 -->
   <joint name="br_steering" type="revolute">
     <origin xyz="-0.1525 0.10997 -0.00127218" rpy="4.22436e-59 -1.37735e-59 0.174533"/>
-    <parent link="body"/>
-    <child link="part_1_3"/>
+    <parent link="base_link"/>
+    <child link="rearsteeringarm_2"/>
     <axis xyz="0 0 1"/>
     <limit effort="10" velocity="10" lower="-0.610865" upper="0.610865"/>
   </joint>
-  <!-- Link part_1_5 -->
-  <link name="part_1_5">
+  <!-- Link frontsteeringarm -->
+  <link name="frontsteeringarm">
     <inertial>
       <origin xyz="0.0160954 1.24761e-09 -0.0207225" rpy="0 0 0"/>
@@ -323,11 +323,11 @@
       <inertia ixx="1.28485e-05" ixy="-1.54012e-13" ixz="1.11198e-06" iyy="1.57606e-05" iyz="1.84212e-12" izz="5.35874e-06"/>
     </inertial>
-    <!-- Part part_1_5 -->
+    <!-- Part frontsteeringarm -->
     <visual>
       <origin xyz="0 0 -0.005" rpy="0 -0 9.24446e-33"/>
       <geometry>
-        <mesh filename="${mesh_dir}/part_1__3.stl"/>
-      </geometry>
-      <material name="part_1_5_material">
+        <mesh filename="${mesh_dir}/frontsteeringarm.stl"/>
+      </geometry>
+      <material name="frontsteeringarm_material">
         <color rgba="0.458824 0.105882 0 1"/>
       </material>
@@ -336,22 +336,22 @@
       <origin xyz="0 0 -0.005" rpy="0 -0 9.24446e-33"/>
       <geometry>
-        <mesh filename="${mesh_dir}/part_1__3.stl"/>
-      </geometry>
-    </collision>
-  </link>
-  <!-- Link part_1_6 -->
-  <link name="part_1_6">
-    <inertial>
-      <origin xyz="-1.47254e-19 3.11998e-18 0.00460287" rpy="0 0 0"/>
+        <mesh filename="${mesh_dir}/frontsteeringarm.stl"/>
+      </geometry>
+    </collision>
+  </link>
+  <!-- Link wheelhub_3 -->
+  <link name="wheelhub_3">
+    <inertial>
+      <origin xyz="-1.47254e-19 3.11997e-18 0.00460287" rpy="0 0 0"/>
       <mass value="0.0820664"/>
       <inertia ixx="3.08808e-05" ixy="0" ixz="-5.47239e-37" iyy="3.08808e-05" iyz="0" izz="5.62507e-05"/>
     </inertial>
-    <!-- Part part_1_6 -->
+    <!-- Part wheelhub_3 -->
     <visual>
       <origin xyz="0 0 -0.005" rpy="-1.5708 -2.15704e-32 0"/>
       <geometry>
-        <mesh filename="${mesh_dir}/part_1__2.stl"/>
-      </geometry>
-      <material name="part_1_6_material">
+        <mesh filename="${mesh_dir}/wheelhub.stl"/>
+      </geometry>
+      <material name="wheelhub_3_material">
         <color rgba="0.498039 0.498039 0.498039 1"/>
       </material>
@@ -360,26 +360,26 @@
       <origin xyz="0 0 -0.005" rpy="-1.5708 -2.15704e-32 0"/>
       <geometry>
-        <mesh filename="${mesh_dir}/part_1__2.stl"/>
-      </geometry>
-    </collision>
-  </link>
-  <!-- Joint from part_1_5 to part_1_6 -->
+        <mesh filename="${mesh_dir}/wheelhub.stl"/>
+      </geometry>
+    </collision>
+  </link>
+  <!-- Joint from frontsteeringarm to wheelhub_3 -->
   <joint name="fl_wheel" type="continuous">
     <origin xyz="-0.005 -2.77556e-17 -0.0433189" rpy="-1.5708 -0 -1.5708"/>
-    <parent link="part_1_5"/>
-    <child link="part_1_6"/>
+    <parent link="frontsteeringarm"/>
+    <child link="wheelhub_3"/>
     <axis xyz="0 0 1"/>
     <limit effort="10" velocity="10"/>
   </joint>
-  <!-- Joint from body to part_1_5 -->
+  <!-- Joint from base_link to frontsteeringarm -->
   <joint name="fl_steering" type="revolute">
     <origin xyz="0.1525 -0.140031 -0.0015" rpy="0 -0 3.14159"/>
-    <parent link="body"/>
-    <child link="part_1_5"/>
+    <parent link="base_link"/>
+    <child link="frontsteeringarm"/>
     <axis xyz="0 0 1"/>
     <limit effort="10" velocity="10" lower="-0.610865" upper="0.610865"/>
   </joint>
-  <!-- Link part_1_7 -->
-  <link name="part_1_7">
+  <!-- Link frontsteeringarm_2 -->
+  <link name="frontsteeringarm_2">
     <inertial>
       <origin xyz="-0.0160954 -1.24761e-09 -0.0207225" rpy="0 0 0"/>
@@ -387,11 +387,11 @@
       <inertia ixx="1.28485e-05" ixy="-1.54012e-13" ixz="-1.11198e-06" iyy="1.57606e-05" iyz="-1.84212e-12" izz="5.35874e-06"/>
     </inertial>
-    <!-- Part part_1_7 -->
+    <!-- Part frontsteeringarm_2 -->
     <visual>
       <origin xyz="0 2.77556e-17 -0.005" rpy="0 -0 3.14159"/>
       <geometry>
-        <mesh filename="${mesh_dir}/part_1__3.stl"/>
-      </geometry>
-      <material name="part_1_7_material">
+        <mesh filename="${mesh_dir}/frontsteeringarm.stl"/>
+      </geometry>
+      <material name="frontsteeringarm_2_material">
         <color rgba="0.458824 0.105882 0 1"/>
       </material>
@@ -400,22 +400,22 @@
       <origin xyz="0 2.77556e-17 -0.005" rpy="0 -0 3.14159"/>
       <geometry>
-        <mesh filename="${mesh_dir}/part_1__3.stl"/>
-      </geometry>
-    </collision>
-  </link>
-  <!-- Link part_1_8 -->
-  <link name="part_1_8">
-    <inertial>
-      <origin xyz="-1.47254e-19 3.11998e-18 0.00460287" rpy="0 0 0"/>
+        <mesh filename="${mesh_dir}/frontsteeringarm.stl"/>
+      </geometry>
+    </collision>
+  </link>
+  <!-- Link wheelhub_4 -->
+  <link name="wheelhub_4">
+    <inertial>
+      <origin xyz="-1.47254e-19 3.11997e-18 0.00460287" rpy="0 0 0"/>
       <mass value="0.0820664"/>
       <inertia ixx="3.08808e-05" ixy="1.05339e-100" ixz="-2.68495e-37" iyy="3.08808e-05" iyz="-3.41845e-68" izz="5.62507e-05"/>
     </inertial>
-    <!-- Part part_1_8 -->
+    <!-- Part wheelhub_4 -->
     <visual>
       <origin xyz="0 0 -0.005" rpy="-1.5708 3.08149e-33 0"/>
       <geometry>
-        <mesh filename="${mesh_dir}/part_1__2.stl"/>
-      </geometry>
-      <material name="part_1_8_material">
+        <mesh filename="${mesh_dir}/wheelhub.stl"/>
+      </geometry>
+      <material name="wheelhub_4_material">
         <color rgba="0.498039 0.498039 0.498039 1"/>
       </material>
@@ -424,38 +424,38 @@
       <origin xyz="0 0 -0.005" rpy="-1.5708 3.08149e-33 0"/>
       <geometry>
-        <mesh filename="${mesh_dir}/part_1__2.stl"/>
-      </geometry>
-    </collision>
-  </link>
-  <!-- Joint from part_1_7 to part_1_8 -->
+        <mesh filename="${mesh_dir}/wheelhub.stl"/>
+      </geometry>
+    </collision>
+  </link>
+  <!-- Joint from frontsteeringarm_2 to wheelhub_4 -->
   <joint name="fr_wheel" type="continuous">
     <origin xyz="0.005 2.77556e-17 -0.0433189" rpy="1.5708 3.93984e-31 -1.5708"/>
-    <parent link="part_1_7"/>
-    <child link="part_1_8"/>
+    <parent link="frontsteeringarm_2"/>
+    <child link="wheelhub_4"/>
     <axis xyz="0 0 1"/>
     <limit effort="10" velocity="10"/>
   </joint>
-  <!-- Joint from body to part_1_7 -->
+  <!-- Joint from base_link to frontsteeringarm_2 -->
   <joint name="fr_steering" type="revolute">
     <origin xyz="-0.1525 -0.140031 -0.0015" rpy="0 -0 -3.14159"/>
-    <parent link="body"/>
-    <child link="part_1_7"/>
+    <parent link="base_link"/>
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