Commit message: Deleted meshes folder and moved everything to URDF

File: perseverance/urdf/rover.urdf (robot description, URDF)
Before this commit: robot perseverance, 11 links, 10 joints
Links:
- link base_link: geometry collision mesh filename=base_link.stl; collision mesh filename=bevel_0_85m_18t_45deg.stl
- link frontsteeringarm: geometry collision mesh filename=frontsteeringarm.stl; visual mesh filename=frontsteeringarm.stl
- link frontsteeringarm_2: geometry collision mesh filename=frontsteeringarm.stl; visual mesh filename=frontsteeringarm.stl
- link rearsteeringarm: geometry collision mesh filename=rearsteeringarm.stl; visual mesh filename=rearsteeringarm.stl
- link rearsteeringarm_2: geometry collision mesh filename=rearsteeringarm.stl; visual mesh filename=rearsteeringarm.stl
- link wheelhub: geometry collision mesh filename=wheelhub.stl; visual mesh filename=wheelhub.stl
- link wheelhub_2: geometry collision mesh filename=wheelhub.stl; visual mesh filename=wheelhub.stl
- link wheelhub_3: geometry collision mesh filename=wheelhub.stl; visual mesh filename=wheelhub.stl
- link wheelhub_4: geometry collision mesh filename=wheelhub.stl; visual mesh filename=wheelhub.stl
- link wheelhub_5: geometry collision mesh filename=wheelhub.stl; visual mesh filename=wheelhub.stl
- link wheelhub_6: geometry collision mesh filename=wheelhub.stl; visual mesh filename=wheelhub.stl

File: perseverance/urdf/rover.urdf.xacro (robot description, xacro)
@@ -2,6 +2,6 @@
 <!-- Generated using onshape-to-robot -->
 <!-- Onshape https://cad.onshape.com/documents/31ca51e87164d5a2ae3b11dc/w/1e07aa3f18f08d453ac8b6a1/e/be108145cc25fea61866c58d -->
-<robot name="perseverance" xmlns:xacro="http://ros.org/wiki/xacro">
-  <xacro:property name="mesh_dir" value="file://$(find perseverance)/meshes"/>
+<robot name="perseverance"
+  xmlns:xacro="http://ros.org/wiki/xacro">
   <!-- Link base_link -->
   <link name="base_link">
@@ -15,5 +15,5 @@
       <origin xyz="-0.15 0.0418583 -0.00306575" rpy="0 -0 -1.5708"/>
       <geometry>
-        <mesh filename="${mesh_dir}/rightbogie.stl"/>
+        <mesh filename="rightbogie.stl"/>
       </geometry>
       <material name="rightbogie_material">
@@ -24,5 +24,5 @@
       <origin xyz="-0.15 0.0418583 -0.00306575" rpy="0 -0 -1.5708"/>
       <geometry>
-        <mesh filename="${mesh_dir}/rightbogie.stl"/>
+        <mesh filename="rightbogie.stl"/>
       </geometry>
     </collision>
@@ -31,5 +31,5 @@
       <origin xyz="-0.012226 -0.042 0.024" rpy="-0 1.5708 0"/>
       <geometry>
-        <mesh filename="${mesh_dir}/bevel_0_85m_18t_45deg.stl"/>
+        <mesh filename="bevel_0_85m_18t_45deg.stl"/>
       </geometry>
       <material name="bevel_0_85m_18t_45deg_material">
@@ -40,5 +40,5 @@
       <origin xyz="-0.012226 -0.042 0.024" rpy="-0 1.5708 0"/>
       <geometry>
-        <mesh filename="${mesh_dir}/bevel_0_85m_18t_45deg.stl"/>
+        <mesh filename="bevel_0_85m_18t_45deg.stl"/>
       </geometry>
     </collision>
@@ -47,5 +47,5 @@
       <origin xyz="0 0 0" rpy="0 -0 0"/>
       <geometry>
-        <mesh filename="${mesh_dir}/base_link.stl"/>
+        <mesh filename="base_link.stl"/>
       </geometry>
       <material name="base_link_material">
@@ -56,5 +56,5 @@
       <origin xyz="0 0 0" rpy="0 -0 0"/>
       <geometry>
-        <mesh filename="${mesh_dir}/base_link.stl"/>
+        <mesh filename="base_link.stl"/>
       </geometry>
     </collision>
@@ -63,5 +63,5 @@
       <origin xyz="0.012226 -0.042 0.024" rpy="-1.3494e-79 -1.5708 0"/>
       <geometry>
-        <mesh filename="${mesh_dir}/bevel_0_85m_18t_45deg.stl"/>
+        <mesh filename="bevel_0_85m_18t_45deg.stl"/>
       </geometry>
       <material name="bevel_0_85m_18t_45deg_2_material">
@@ -72,5 +72,5 @@
       <origin xyz="0.012226 -0.042 0.024" rpy="-1.3494e-79 -1.5708 0"/>
       <geometry>
-        <mesh filename="${mesh_dir}/bevel_0_85m_18t_45deg.stl"/>
+        <mesh filename="bevel_0_85m_18t_45deg.stl"/>
       </geometry>
     </collision>
@@ -79,5 +79,5 @@
       <origin xyz="-0.1425 -0.140031 0.043" rpy="3.14159 -0 -3.14159"/>
       <geometry>
-        <mesh filename="${mesh_dir}/mg995.stl"/>
+        <mesh filename="mg995.stl"/>
       </geometry>
       <material name="mg995_material">
@@ -88,5 +88,5 @@
       <origin xyz="-0.1425 -0.140031 0.043" rpy="3.14159 -0 -3.14159"/>
       <geometry>
-        <mesh filename="${mesh_dir}/mg995.stl"/>
+        <mesh filename="mg995.stl"/>
       </geometry>
     </collision>
@@ -95,5 +95,5 @@
       <origin xyz="-0.150764 0.100122 0.0432278" rpy="3.14159 -0 1.74533"/>
       <geometry>
-        <mesh filename="${mesh_dir}/mg995.stl"/>
+        <mesh filename="mg995.stl"/>
       </geometry>
       <material name="mg995_2_material">
@@ -104,5 +104,5 @@
       <origin xyz="-0.150764 0.100122 0.0432278" rpy="3.14159 -0 1.74533"/>
       <geometry>
-        <mesh filename="${mesh_dir}/mg995.stl"/>
+        <mesh filename="mg995.stl"/>
       </geometry>
     </collision>
@@ -111,5 +111,5 @@
       <origin xyz="0.1425 -0.140031 0.043" rpy="3.14159 -0 -2.01228e-16"/>
       <geometry>
-        <mesh filename="${mesh_dir}/mg995.stl"/>
+        <mesh filename="mg995.stl"/>
       </geometry>
       <material name="mg995_3_material">
@@ -120,5 +120,5 @@
       <origin xyz="0.1425 -0.140031 0.043" rpy="3.14159 -0 -2.01228e-16"/>
       <geometry>
-        <mesh filename="${mesh_dir}/mg995.stl"/>
+        <mesh filename="mg995.stl"/>
       </geometry>
     </collision>
@@ -127,5 +127,5 @@
       <origin xyz="0.115 -0.042 0.024" rpy="0 -0 -1.5708"/>
       <geometry>
-        <mesh filename="${mesh_dir}/leftrocker.stl"/>
+        <mesh filename="leftrocker.stl"/>
       </geometry>
       <material name="leftrocker_material">
@@ -136,5 +136,5 @@
       <origin xyz="0.115 -0.042 0.024" rpy="0 -0 -1.5708"/>
       <geometry>
-        <mesh filename="${mesh_dir}/leftrocker.stl"/>
+        <mesh filename="leftrocker.stl"/>
       </geometry>
     </collision>
@@ -143,5 +143,5 @@
       <origin xyz="-0.115 -0.042 0.024" rpy="0 -0 -1.5708"/>
       <geometry>
-        <mesh filename="${mesh_dir}/rightrocker.stl"/>
+        <mesh filename="rightrocker.stl"/>
       </geometry>
       <material name="rightrocker_material">
@@ -152,5 +152,5 @@
       <origin xyz="-0.115 -0.042 0.024" rpy="0 -0 -1.5708"/>
       <geometry>
-        <mesh filename="${mesh_dir}/rightrocker.stl"/>
+        <mesh filename="rightrocker.stl"/>
       </geometry>
     </collision>
@@ -159,5 +159,5 @@
       <origin xyz="0.150764 0.100122 0.0432278" rpy="3.14159 -0 1.39626"/>
       <geometry>
-        <mesh filename="${mesh_dir}/mg995.stl"/>
+        <mesh filename="mg995.stl"/>
       </geometry>
       <material name="mg995_4_material">
@@ -168,5 +168,5 @@
       <origin xyz="0.150764 0.100122 0.0432278" rpy="3.14159 -0 1.39626"/>
       <geometry>
-        <mesh filename="${mesh_dir}/mg995.stl"/>
+        <mesh filename="mg995.stl"/>
       </geometry>
     </collision>
@@ -175,5 +175,5 @@
       <origin xyz="0.15 0.0418583 -0.00306575" rpy="0 -0 -1.5708"/>
       <geometry>
-        <mesh filename="${mesh_dir}/leftbogie.stl"/>
+        <mesh filename="leftbogie.stl"/>
       </geometry>
       <material name="leftbogie_material">
@@ -184,5 +184,5 @@
       <origin xyz="0.15 0.0418583 -0.00306575" rpy="0 -0 -1.5708"/>
       <geometry>
-        <mesh filename="${mesh_dir}/leftbogie.stl"/>
+        <mesh filename="leftbogie.stl"/>
       </geometry>
     </collision>
@@ -199,5 +199,5 @@
       <origin xyz="2.77556e-17 2.77556e-17 -0.005" rpy="9.24446e-33 -2.82529e-32 -4.77087e-18"/>
       <geometry>
-        <mesh filename="${mesh_dir}/rearsteeringarm.stl"/>
+        <mesh filename="rearsteeringarm.stl"/>
       </geometry>
       <material name="rearsteeringarm_material">
@@ -208,5 +208,5 @@
       <origin xyz="2.77556e-17 2.77556e-17 -0.005" rpy="9.24446e-33 -2.82529e-32 -4.77087e-18"/>
       <geometry>
-        <mesh filename="${mesh_dir}/rearsteeringarm.stl"/>
+        <mesh filename="rearsteeringarm.stl"/>
       </geometry>
     </collision>
@@ -223,5 +223,5 @@
       <origin xyz="0 0 -0.005" rpy="-1.5708 1.35456e-17 3.31859e-65"/>
       <geometry>
-        <mesh filename="${mesh_dir}/wheelhub.stl"/>
+        <mesh filename="wheelhub.stl"/>
       </geometry>
       <material name="wheelhub_material">
@@ -232,5 +232,5 @@
       <origin xyz="0 0 -0.005" rpy="-1.5708 1.35456e-17 3.31859e-65"/>
       <geometry>
-        <mesh filename="${mesh_dir}/wheelhub.stl"/>
+        <mesh filename="wheelhub.stl"/>
       </geometry>
     </collision>
@@ -263,5 +263,5 @@
       <origin xyz="2.77556e-17 2.77556e-17 -0.005" rpy="-8.84344e-75 -0 -7.75341e-18"/>
       <geometry>
-        <mesh filename="${mesh_dir}/rearsteeringarm.stl"/>
+        <mesh filename="rearsteeringarm.stl"/>
       </geometry>
       <material name="rearsteeringarm_2_material">
@@ -272,5 +272,5 @@
       <origin xyz="2.77556e-17 2.77556e-17 -0.005" rpy="-8.84344e-75 -0 -7.75341e-18"/>
       <geometry>
-        <mesh filename="${mesh_dir}/rearsteeringarm.stl"/>
+        <mesh filename="rearsteeringarm.stl"/>
       </geometry>
     </collision>
@@ -287,5 +287,5 @@
       <origin xyz="2.77556e-17 0 -0.005" rpy="-1.5708 1.93111e-18 9.91647e-75"/>
       <geometry>
-        <mesh filename="${mesh_dir}/wheelhub.stl"/>
+        <mesh filename="wheelhub.stl"/>
       </geometry>
       <material name="wheelhub_2_material">
@@ -296,5 +296,5 @@
       <origin xyz="2.77556e-17 0 -0.005" rpy="-1.5708 1.93111e-18 9.91647e-75"/>
       <geometry>
-        <mesh filename="${mesh_dir}/wheelhub.stl"/>
+        <mesh filename="wheelhub.stl"/>
       </geometry>
     </collision>
@@ -327,5 +327,5 @@
       <origin xyz="0 0 -0.005" rpy="0 -0 9.24446e-33"/>
       <geometry>
-        <mesh filename="${mesh_dir}/frontsteeringarm.stl"/>
+        <mesh filename="frontsteeringarm.stl"/>
       </geometry>
       <material name="frontsteeringarm_material">
@@ -336,5 +336,5 @@
       <origin xyz="0 0 -0.005" rpy="0 -0 9.24446e-33"/>
       <geometry>
-        <mesh filename="${mesh_dir}/frontsteeringarm.stl"/>
+        <mesh filename="frontsteeringarm.stl"/>
       </geometry>
     </collision>
@@ -351,5 +351,5 @@
       <origin xyz="0 0 -0.005" rpy="-1.5708 -2.15704e-32 0"/>
       <geometry>
-        <mesh filename="${mesh_dir}/wheelhub.stl"/>
+        <mesh filename="wheelhub.stl"/>
       </geometry>
       <material name="wheelhub_3_material">
@@ -360,5 +360,5 @@
       <origin xyz="0 0 -0.005" rpy="-1.5708 -2.15704e-32 0"/>
       <geometry>
-        <mesh filename="${mesh_dir}/wheelhub.stl"/>
+        <mesh filename="wheelhub.stl"/>
       </geometry>
     </collision>
@@ -391,5 +391,5 @@
       <origin xyz="0 2.77556e-17 -0.005" rpy="0 -0 3.14159"/>
       <geometry>
-        <mesh filename="${mesh_dir}/frontsteeringarm.stl"/>
+        <mesh filename="frontsteeringarm.stl"/>
       </geometry>
       <material name="frontsteeringarm_2_material">
@@ -400,5 +400,5 @@
       <origin xyz="0 2.77556e-17 -0.005" rpy="0 -0 3.14159"/>
       <geometry>
-        <mesh filename="${mesh_dir}/frontsteeringarm.stl"/>
+        <mesh filename="frontsteeringarm.stl"/>
       </geometry>
     </collision>
@@ -415,5 +415,5 @@
       <origin xyz="0 0 -0.005" rpy="-1.5708 3.08149e-33 0"/>
       <geometry>
-        <mesh filename="${mesh_dir}/wheelhub.stl"/>
+        <mesh filename="wheelhub.stl"/>
       </geometry>
       <material name="wheelhub_4_material">
@@ -424,5 +424,5 @@
       <origin xyz="0 0 -0.005" rpy="-1.5708 3.08149e-33 0"/>
       <geometry>
-        <mesh filename="${mesh_dir}/wheelhub.stl"/>
+        <mesh filename="wheelhub.stl"/>
       </geometry>
     </collision>
@@ -455,5 +455,5 @@
       <origin xyz="0 0 -0.005" rpy="-1.5708 -4.31408e-32 0"/>
       <geometry>
-        <mesh filename="${mesh_dir}/wheelhub.stl"/>
+        <mesh filename="wheelhub.stl"/>
       </geometry>
       <material name="wheelhub_5_material">
@@ -464,5 +464,5 @@
       <origin xyz="0 0 -0.005" rpy="-1.5708 -4.31408e-32 0"/>
       <geometry>
-        <mesh filename="${mesh_dir}/wheelhub.stl"/>
+        <mesh filename="wheelhub.stl"/>
       </geometry>
     </collision>
@@ -487,5 +487,5 @@
       <origin xyz="1.73472e-18 -6.93889e-18 -0.01" rpy="-1.5708 -1.11022e-15 0"/>
       <geometry>
-        <mesh filename="${mesh_dir}/wheelhub.stl"/>
+        <mesh filename="wheelhub.stl"/>
       </geometry>
       <material name="wheelhub_6_material">
@@ -496,5 +496,5 @@
       <origin xyz="1.73472e-18 -6.93889e-18 -0.01" rpy="-1.5708 -1.11022e-15 0"/>
       <geometry>
-        <mesh filename="${mesh_dir}/wheelhub.stl"/>
+        <mesh filename="wheelhub.stl"/>
       </geometry>
     </collision>

Commit message: Updating files

File: perseverance/urdf/rover.urdf (robot description, URDF)
Before this commit: robot perseverance, 11 links, 10 joints
Links:
- link base_link: mass 1.16655 -> 0.946692
Joints:
- joint bl_steering: origin xyz=0.1525 0.10997 -0.00127218 rpy=-1.249e-16 4.18641e-16 2.96706 -> xyz=0.1025 0.10997 -0.00127218 rpy=-1.249e-16 4.18641e-16 2.96706
- joint bl_wheel: origin xyz=-0.005 -5.55112e-17 -0.0463814 rpy=-1.5708 1.249e-16 -1.5708 -> xyz=-0.005 2.77556e-17 -0.0463814 rpy=-1.5708 1.249e-16 -1.5708
- joint fl_steering: origin xyz=0.1525 -0.140031 -0.0015 rpy=0 -0 3.14159 -> xyz=0.1025 -0.140031 -0.0015 rpy=0 -0 3.14159
- joint fl_wheel: origin xyz=-0.005 -2.77556e-17 -0.0433189 rpy=-1.5708 -0 -1.5708 -> xyz=-0.005 2.77556e-17 -0.0433189 rpy=-1.5708 -0 -1.5708
- joint ml_wheel: origin xyz=0.172 -0.00814152 -0.0476535 rpy=1.5708 -0 -1.5708 -> xyz=0.122 -0.00814152 -0.0476535 rpy=1.5708 -0 -1.5708

Commit message: Fixed script

File: perseverance/urdf/rover.urdf (robot description, URDF)
Before this commit: robot perseverance, 11 links, 10 joints
Links:
- link base_link: mass 0.946692 -> 0.946932

Commit message: Fixing generation tool and applying automated edits to urdf

File: perseverance/urdf/rover.urdf (robot description, URDF)
Before this commit: robot perseverance, 11 links, 10 joints
Links:
- removed link wheelhub
- removed link wheelhub_2
- removed link wheelhub_3
- removed link wheelhub_4
- removed link wheelhub_5
- removed link wheelhub_6
- added link base_footprint
- added link wheel, mass 0.0820664; collision mesh filename=package://perseverance/urdf/wheel.stl; visual mesh filename=package://perseverance/urdf/wheel.stl
- added link wheel_2, mass 0.0820664; collision mesh filename=package://perseverance/urdf/wheel.stl; visual mesh filename=package://perseverance/urdf/wheel.stl
- added link wheel_3, mass 0.0820664; collision mesh filename=package://perseverance/urdf/wheel.stl; visual mesh filename=package://perseverance/urdf/wheel.stl
- added link wheel_4, mass 0.0820664; collision mesh filename=package://perseverance/urdf/wheel.stl; visual mesh filename=package://perseverance/urdf/wheel.stl
- added link wheel_5, mass 0.0820664; collision mesh filename=package://perseverance/urdf/wheel.stl; visual mesh filename=package://perseverance/urdf/wheel.stl
- added link wheel_6, mass 0.0820664; collision mesh filename=package://perseverance/urdf/wheel.stl; visual mesh filename=package://perseverance/urdf/wheel.stl
- link base_link: mass 0.946932 -> 1.18472; geometry collision mesh filename=package://perseverance/urdf/base_link.stl; collision mesh filename=package://perseverance/urdf/bevel_0_85m_18t_45deg.stl
- link frontsteeringarm: mass 0.0305721 -> 0.0304253; geometry collision mesh filename=package://perseverance/urdf/frontsteeringarm.stl; visual mesh filename=package://perseverance/urdf/frontsteeringarm.stl
- link frontsteeringarm_2: mass 0.0305721 -> 0.0304253; geometry collision mesh filename=package://perseverance/urdf/frontsteeringarm.stl; visual mesh filename=package://perseverance/urdf/frontsteeringarm.stl
- link rearsteeringarm: mass 0.0309807 -> 0.0308339; geometry collision mesh filename=package://perseverance/urdf/rearsteeringarm.stl; visual mesh filename=package://perseverance/urdf/rearsteeringarm.stl
- link rearsteeringarm_2: mass 0.0309807 -> 0.0308339; geometry collision mesh filename=package://perseverance/urdf/rearsteeringarm.stl; visual mesh filename=package://perseverance/urdf/rearsteeringarm.stl
Joints:
- added joint base_footprint_to_base_link: type fixed, parent base_footprint, child base_link, origin xyz=-0.015030 0.025000 0.000000 rpy=0.000000 0.000000 1.570796
- joint bl_steering: limit lower=-0.610865 upper=0.610865 effort=10 velocity=10 -> lower=-0.785398 upper=0.436332 effort=10 velocity=10; origin xyz=0.1025 0.10997 -0.00127218 rpy=-1.249e-16 4.18641e-16 2.96706 -> xyz=0.1025 0.10997 -0.00127218 rpy=-1.249e-16 4.18641e-16 3.141593
- joint bl_wheel: child wheelhub -> wheel
- joint br_steering: limit lower=-0.610865 upper=0.610865 effort=10 velocity=10 -> lower=-0.436332 upper=0.785398 effort=10 velocity=10; origin xyz=-0.1525 0.10997 -0.00127218 rpy=4.22436e-59 -1.37735e-59 0.174533 -> xyz=-0.1525 0.10997 -0.00127218 rpy=4.22436e-59 -1.37735e-59 0.000000
- joint br_wheel: child wheelhub_2 -> wheel_2
- joint fl_wheel: child wheelhub_3 -> wheel_3
- joint fr_wheel: child wheelhub_4 -> wheel_4
- joint ml_wheel: child wheelhub_6 -> wheel_6
- joint mr_wheel: child wheelhub_5 -> wheel_5

Commit message: Updated URDF

File: perseverance/urdf/rover.urdf (robot description, URDF)
Before this commit: robot perseverance, 12 links, 11 joints
Links:
- removed link base_footprint
- added link base_link_centered
Joints:
- removed joint base_footprint_to_base_link
- added joint base_link_centered_to_base_link: type fixed, parent base_link_centered, child base_link, origin xyz=-0.015030 0.025000 0.000000 rpy=0.000000 0.000000 1.570796

Commit message: Updated steering limits and automatically update config file

File: perseverance/urdf/rover.urdf (robot description, URDF)
Before this commit: robot perseverance, 12 links, 11 joints
Joints:
- joint bl_steering: limit lower=-0.785398 upper=0.436332 effort=10 velocity=10 -> lower=-0.610865 upper=0.610865 effort=10 velocity=10
- joint br_steering: limit lower=-0.436332 upper=0.785398 effort=10 velocity=10 -> lower=-0.610865 upper=0.610865 effort=10 velocity=10
